Commit message: add lidar and d435 link and turn off rviz to run on robot

File: omni_description/urdf/omni.urdf.xacro (robot description, xacro)
@@ -17,14 +17,18 @@
     </link>
     <!--CAM D435-->
-    <xacro:sensor_d435 name="realsense_d435" parent="base_link">
+    <joint name="lidar_joint" type="fixed">
+        <parent link="base_link"/>
+        <child link="camera_link"/>
         <origin xyz="${d435_x} 0 ${d435_z}" rpy="0 0 0"/>
-    </xacro:sensor_d435>
+    </joint>
+    <link name="camera_link">
+    </link>
     <!--LIDAR-->
     <joint name="lidar_joint" type="fixed">
         <parent link="base_link"/>
-        <child link="lidar_link"/>
+        <child link="laser"/>
         <origin xyz="0 0 ${lidar_z}" rpy="0 0 0"/>
     </joint>
-    <link name="lidar_link">
+    <link name="laser">
     </link>
 </robot>

Commit message: fix urdf error and change frame in rtabmap

File: omni_description/urdf/omni.urdf.xacro (robot description, xacro)
@@ -17,5 +17,5 @@
     </link>
     <!--CAM D435-->
-    <joint name="lidar_joint" type="fixed">
+    <joint name="camera_joint" type="fixed">
         <parent link="base_link"/>
         <child link="camera_link"/>

Commit message: add imu to description

File: omni_description/urdf/omni.urdf.xacro (robot description, xacro)
@@ -8,4 +8,5 @@
     <xacro:property name="d435_x" value="0.115"/>
     <xacro:property name="lidar_z" value="0.34"/>
+    <xacro:property name="imu_z" value="0.13"/>
     <link name="base_footprint"/>
     <joint name="base_joint" type="fixed">
@@ -32,3 +33,11 @@
     <link name="laser">
     </link>
+    <!--IMU-->
+    <joint name="imu_joint" type="fixed">
+        <parent link="base_link"/>
+        <child link="imu"/>
+        <origin xyz="0 0 ${imu_z}" rpy="0 0 0"/>
+    </joint>
+    <link name="imu">
+    </link>
 </robot>
